File: BBBCanFly.sch (KiCad schematic (older format))
At the start: 0 parts

Commit message: sch has been finished
Changed lines of the file:
@@
 EESchema Schematic File Version 2
+LIBS:BBBCanFly-rescue
 LIBS:power
 LIBS:device
@@
 F0 "power" 60
 F1 "power.sch" 60
+F2 "24V" O R 8500 4300 60
 $EndSheet
 $Sheet
@@
 F0 "interface" 60
 F1 "interface.sch" 60
+F2 "24V" I L 9100 4300 60
 $EndSheet
+Wire Wire Line
+	9100 4300 8500 4300
 $EndSCHEMATC
